Commit message: chore: remove redundant tags and parameters from mate_p1w configuration
Remove unnecessary <axis> and <limit> tags that were automatically
generated but are not required for fixed joints.

File: robots/mate_p1w_description/urdf/mate_p1w.urdf (robot description, URDF)
Before this commit: robot mate_p1w, 51 links, 50 joints
Links:
- link base_link: mass 0.0 -> None
Joints:
- joint base_to_mobile_base_joint: axis 1.0 0.0 0.0 -> (none); limit lower=-3.14 upper=3.14 effort=0.0 velocity=0.0 -> (none)
- joint left_forearm_cover_joint: axis 1.0 0.0 0.0 -> (none); limit lower=-3.14 upper=3.14 effort=0.0 velocity=0.0 -> (none)
- joint left_front_wheel_cover_joint: axis 0.0 1.0 0.0 -> (none)
- joint left_head_joint: axis 1.0 0.0 0.0 -> (none); limit lower=-3.14 upper=3.14 effort=0.0 velocity=0.0 -> (none)
- joint left_rear_wheel_cover_joint: axis 0.0 1.0 0.0 -> (none); limit lower=-3.14 upper=3.14 effort=0.0 velocity=0.0 -> (none)
- joint left_shoulder_cap_joint: axis 1.0 0.0 0.0 -> (none); limit lower=-3.14 upper=3.14 effort=0.0 velocity=0.0 -> (none)
- joint left_shoulder_cover_joint: axis 1.0 0.0 0.0 -> (none); limit lower=-3.14 upper=3.14 effort=0.0 velocity=0.0 -> (none)
- joint mobile_base_cover_joint: axis 1.0 0.0 0.0 -> (none); limit lower=-3.14 upper=3.14 effort=0.0 velocity=0.0 -> (none)
- joint mobile_base_to_body_joint: axis 1.0 0.0 0.0 -> (none); limit lower=-3.14 upper=3.14 effort=0.0 velocity=0.0 -> (none)
- joint neck_joint: axis 1.0 0.0 0.0 -> (none); limit lower=-3.14 upper=3.14 effort=0.0 velocity=0.0 -> (none)
- joint pelvis_joint: axis 1.0 0.0 0.0 -> (none); limit lower=-3.14 upper=3.14 effort=0.0 velocity=0.0 -> (none)
- joint right_forearm_cover_joint: axis 1.0 0.0 0.0 -> (none); limit lower=-3.14 upper=3.14 effort=0.0 velocity=0.0 -> (none)
- joint right_front_wheel_cover_joint: axis 0.0 1.0 0.0 -> (none)
- joint right_head_joint: axis 1.0 0.0 0.0 -> (none); limit lower=-3.14 upper=3.14 effort=0.0 velocity=0.0 -> (none)
- joint right_rear_wheel_cover_joint: axis 0.0 1.0 0.0 -> (none); limit lower=-3.14 upper=3.14 effort=0.0 velocity=0.0 -> (none)
- joint right_shoulder_cap_joint: axis 1.0 0.0 0.0 -> (none); limit lower=-3.14 upper=3.14 effort=0.0 velocity=0.0 -> (none)
- joint right_shoulder_cover_joint: axis 1.0 0.0 0.0 -> (none); limit lower=-3.14 upper=3.14 effort=0.0 velocity=0.0 -> (none)
- joint upper_body_joint: axis 1.0 0.0 0.0 -> (none); limit lower=-3.14 upper=3.14 effort=0.0 velocity=0.0 -> (none)
