Commit message: Update README.md and Rename SB1_Core to sb1_core_description: Unify lowercase naming throughout package

File: robots/sb1_core_description/urdf/sb1_core.urdf (robot description, URDF)
Before this commit: robot SB1_Core, 34 links, 33 joints
Links:
- link base_bottom_plate: geometry collision mesh filename=package://sb1_core_description/meshes/base_bottom_plate.stl; visual mesh filename=package://sb1_core_description/meshes/base_bottom_plate.stl
- link base_cover: geometry collision mesh filename=package://sb1_core_description/meshes/base_cover.stl; visual mesh filename=package://sb1_core_description/meshes/base_cover.stl
- link base_slot_track_rail: geometry collision mesh filename=package://sb1_core_description/meshes/base_slot_track_rail.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; visual mesh filename=package://sb1_core_description/meshes/base_slot_track_rail.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
- link base_top_plate: geometry collision mesh filename=package://sb1_core_description/meshes/base_top_plate.stl; visual mesh filename=package://sb1_core_description/meshes/base_top_plate.stl
- link camera_d435_housing: geometry collision mesh filename=package://sb1_core_description/meshes/camera_d435_housing.s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; visual mesh filename=package://sb1_core_description/meshes/camera_d435_housing.s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
- link camera_d435_sensor: geometry collision mesh filename=package://sb1_core_description/meshes/camera_d435_sensor.stl; visual mesh filename=package://sb1_core_description/meshes/camera_d435_sensor.stl
- link front_left_emergency_button: geometry collision mesh filename=package://sb1_core_description/meshes/front_left_emergency_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; visual mesh filename=package://sb1_core_description/meshes/front_left_emergency_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
- link front_left_emergency_button_base: geometry collision mesh filename=package://sb1_core_description/meshes/front_left_emergency_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; visual mesh filename=package://sb1_core_description/meshes/front_left_emergency_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
- link front_left_swerve_unit: geometry collision mesh filename=package://sb1_core_description/meshes/front_left_swerve_uni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; visual mesh filename=package://sb1_core_description/meshes/front_left_swerve_uni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
- link front_left_wheel_cover: geometry collision mesh filename=package://sb1_core_description/meshes/front_left_wheel_cove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; visual mesh filename=package://sb1_core_description/meshes/front_left_wheel_cove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
- link front_left_wheel_motor: geometry collision mesh filename=package://sb1_core_description/meshes/front_left_wheel_moto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; visual mesh filename=package://sb1_core_description/meshes/front_left_wheel_moto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
- link front_left_wheel_tire: geometry collision mesh filename=package://sb1_core_description/meshes/front_left_wheel_tire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; visual mesh filename=package://sb1_core_description/meshes/front_left_wheel_tire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
- link front_mid360_base: geometry collision mesh filename=package://sb1_core_description/meshes/mid360_base.stl; visual mesh filename=package://sb1_core_description/meshes/mid360_base.stl
- link front_mid360_cover: geometry collision mesh filename=package://sb1_core_description/meshes/mid360_cover.stl; visual mesh filename=package://sb1_core_description/meshes/mid360_cover.stl
- link front_mid360_sensor: geometry collision mesh filename=package://sb1_core_description/meshes/mid360_sensor.stl; visual mesh filename=package://sb1_core_description/meshes/mid360_sensor.stl
- link front_right_emergency_button: geometry collision mesh filename=package://sb1_core_description/meshes/front_right_emergency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; visual mesh filename=package://sb1_core_description/meshes/front_right_emergency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
- link front_right_emergency_button_base: geometry collision mesh filename=package://sb1_core_description/meshes/front_right_emergency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; visual mesh filename=package://sb1_core_description/meshes/front_right_emergency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
- link front_right_swerve_unit: geometry collision mesh filename=package://sb1_core_description/meshes/front_right_swerve_un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; visual mesh filename=package://sb1_core_description/meshes/front_right_swerve_un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
- link front_right_wheel_cover: geometry collision mesh filename=package://sb1_core_description/meshes/front_right_wheel_cov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; visual mesh filename=package://sb1_core_description/meshes/front_right_wheel_cov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
- link front_right_wheel_motor: geometry collision mesh filename=package://sb1_core_description/meshes/front_right_wheel_mot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; visual mesh filename=package://sb1_core_description/meshes/front_right_wheel_mot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
- link front_right_wheel_tire: geometry collision mesh filename=package://sb1_core_description/meshes/front_right_wheel_tir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; visual mesh filename=package://sb1_core_description/meshes/front_right_wheel_tir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
- link rear_left_swerve_unit: geometry collision mesh filename=package://sb1_core_description/meshes/rear_left_swerve_unit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; visual mesh filename=package://sb1_core_description/meshes/rear_left_swerve_unit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
- link rear_left_wheel_cover: geometry collision mesh filename=package://sb1_core_description/meshes/rear_left_wheel_cover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; visual mesh filename=package://sb1_core_description/meshes/rear_left_wheel_cover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
- link rear_left_wheel_motor: geometry collision mesh filename=package://sb1_core_description/meshes/rear_left_wheel_motor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; visual mesh filename=package://sb1_core_description/meshes/rear_left_wheel_motor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
- link rear_left_wheel_tire: geometry collision mesh filename=package://sb1_core_description/meshes/rear_left_wheel_tire.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; visual mesh filename=package://sb1_core_description/meshes/rear_left_wheel_tire.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
- link rear_mid360_base: geometry collision mesh filename=package://sb1_core_description/meshes/mid360_base.stl; visual mesh filename=package://sb1_core_description/meshes/mid360_base.stl
- link rear_mid360_cover: geometry collision mesh filename=package://sb1_core_description/meshes/mid360_cover.stl; visual mesh filename=package://sb1_core_description/meshes/mid360_cover.stl
- link rear_mid360_sensor: geometry collision mesh filename=package://sb1_core_description/meshes/mid360_sensor.stl; visual mesh filename=package://sb1_core_description/meshes/mid360_sensor.stl
- link rear_right_swerve_unit: geometry collision mesh filename=package://sb1_core_description/meshes/rear_right_swerve_uni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; visual mesh filename=package://sb1_core_description/meshes/rear_right_swerve_uni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
- link rear_right_wheel_cover: geometry collision mesh filename=package://sb1_core_description/meshes/rear_right_wheel_cove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; visual mesh filename=package://sb1_core_description/meshes/rear_right_wheel_cove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
- link rear_right_wheel_motor: geometry collision mesh filename=package://sb1_core_description/meshes/rear_right_wheel_moto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; visual mesh filename=package://sb1_core_description/meshes/rear_right_wheel_moto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
- link rear_right_wheel_tire: geometry collision mesh filename=package://sb1_core_description/meshes/rear_right_wheel_tire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; visual mesh filename=package://sb1_core_description/meshes/rear_right_wheel_tire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
- link speaker: geometry collision mesh filename=package://sb1_core_description/meshes/speaker.stl; visual mesh filename=package://sb1_core_description/meshes/speaker.stl
