Commit message: Validate worker URDF and add visualization assets

File: robots/agirobots_worker_description/urdf/agirobots_worker.urdf (robot description, URDF)
Before this commit: robot AGIRobots Worker, 123 links, 122 joints
Joints:
- joint upper_body_upper_right_cover_joint: limit lower=-0.3 upper=2.5 -> lower=-0.3 upper=2.5 effort=0 velocity=0
